Commit message: add /angle_cmd plugin

File: urdf/pan_tilt.xacro (robot description, xacro)
@@ -17,5 +17,5 @@
                 <cylinder radius="${base_link_radius}" length="${base_link_length}"/>
             </geometry>
-            <origin xyz="0.0 0.0 0.015" rpy="0.0 0.0 0.0"/>
+            <origin xyz="0.0 0.0 0.30" rpy="0.0 0.0 0.0"/>
         </visual>
         <collision>
@@ -23,5 +23,5 @@
                 <cylinder radius="${base_link_radius}" length="${base_link_length}"/>
             </geometry>
-            <origin xyz="0.0 0.0 0.015" rpy="0.0 0.0 0.0"/>
+            <origin xyz="0.0 0.0 0.30" rpy="0.0 0.0 0.0"/>
         </collision>
         <inertial>
@@ -33,8 +33,8 @@
         <parent link="base_link"/>
         <child link="pan_link"/>
-        <origin xyz="0.0 0.0 0.015"/>
+        <origin xyz="0.0 0.0 0.315"/>
         <axis xyz="0.0 0.0 1.0"/>
      --  <limit lower="-1000000" upper="1000000" effort="300" velocity="0.1"/>
-        <dynamics damping="1" friction="1"/>
+        <dynamics damping="50" friction="1"/>
     </joint>
     <link name="pan_link">
@@ -64,6 +64,6 @@
         <origin xyz="0.0 0.09 1.5"/>
         <axis xyz="0.0 1.0 0.0"/>
-       <limit lower="-2.0" upper="2.0" effort="300.0" velocity="0.5"/>
-        <dynamics damping="1" friction="1"/>
+       <limit lower="-1000000" upper="1000000" effort="300.0" velocity="0.5"/>
+        <dynamics damping="50" friction="1"/>
     </joint>
     <link name="tilt_link">
@@ -240,5 +240,5 @@
           <horizontal_fov>1.487020523</horizontal_fov>
           <image>
-            <width>680</width>
+            <width>640</width>
             <height>480</height>
           </image>
@@ -255,5 +255,5 @@
         <always_on>1</always_on>
         <update_rate>90</update_rate>
-        <visualize>0</visualize>
+        <visualize>1</visualize>
       </sensor>
     </gazebo>
@@ -283,5 +283,6 @@
         <pointCloudCutoffMax>9.0</pointCloudCutoffMax>
       </plugin>
-      <plugin name="my_robot" filename="libmyrobot_plugin.so"/>
-    </gazebo>
+     <plugin name="my_pantilt" filename="libmypantilt_plugin.so"/>
+     <plugin name="my_robot" filename="libmyrobot_plugin.so"/>
+</gazebo>
 </robot>

Commit message: -

File: urdf/pan_tilt.xacro (robot description, xacro)
@@ -11,4 +11,5 @@
         <parent link="world"/>
         <child link="base_link"/>
+        <static>0</static>
     </joint>
     <link name="base_link">
@@ -23,5 +24,5 @@
                 <cylinder radius="${base_link_radius}" length="${base_link_length}"/>
             </geometry>
-            <origin xyz="0.0 0.0 0.30" rpy="0.0 0.0 0.0"/>
+           <origin xyz="0.0 0.0 0.30" rpy="0.0 0.0 0.0"/>
         </collision>
         <inertial>
@@ -170,4 +171,15 @@
     <link name="camera_color_optical_frame"/>
     <gazebo reference="camera_link">
+     <self_collide>0</self_collide>
+      <enable_wind>0</enable_wind>
+      <kinematic>0</kinematic>
+      <gravity>0</gravity>
+      <!--<mu>1</mu>-->
+      <mu2>1</mu2>
+      <fdir1>0 0 0</fdir1>
+      <!--<slip1>0</slip1>
+      <slip2>0</slip2>-->
+      <kp>1e+13</kp>
+      <kd>1</kd>
       <sensor name="cameracolor" type="camera">
         <camera name="camera">

Commit message: added pan-tilt plugin code

File: urdf/pan_tilt.xacro (robot description, xacro)
@@ -18,5 +18,5 @@
                 <cylinder radius="${base_link_radius}" length="${base_link_length}"/>
             </geometry>
-            <origin xyz="0.0 0.0 0.30" rpy="0.0 0.0 0.0"/>
+          <origin xyz="0.0 0.0 0.30" rpy="0.0 0.0 0.0"/>
         </visual>
         <collision>
@@ -36,5 +36,5 @@
         <origin xyz="0.0 0.0 0.315"/>
         <axis xyz="0.0 0.0 1.0"/>
-     --  <limit lower="-1000000" upper="1000000" effort="300" velocity="0.1"/>
+       <limit lower="-1000000" upper="1000000" effort="300" velocity="0.1"/>
         <dynamics damping="50" friction="1"/>
     </joint>
@@ -90,5 +90,5 @@
     </link>
     <joint name="camera_joint" type="fixed">
-      <origin xyz="0.0 0.04 0.22" rpy="3.141592 -1.5707 0.0"/>
+      <origin xyz="0.0 0.0 0.22" rpy="0 -1.5707 0.0"/>
       <parent link="tilt_link"/>
       <child link="camera_bottom_screw_frame" />
@@ -272,6 +272,6 @@
     <gazebo>
     <plugin name="gazebo_api" filename="libgazebo_ros_api_plugin.so"/>
-    <plugin name="my_pantilt" filename="libmypantilt_plugin.so"/>
-     <plugin name="my_robot" filename="libmyrobot_plugin.so"/>
+    <plugin name="my_pantilt2" filename="libmypantilt2_plugin.so"/>
+    <plugin name="my_pantilt1" filename="libmypantilt1_plugin.so"/>
     <plugin name="camera" filename="librealsense_gazebo_plugin.so">
         <prefix>camera</prefix>
